Commit message: Added tennis racquet files and hopefully added in racquet link

File: mmp_panda.urdf (robot description, URDF)
Before this commit: robot mmp_panda, 11 links, 10 joints
Links:
- added link racquetlink, mass .3203496; visual mesh filename=../../../cs225a/CS225a_TennisBot/Objects/Visual/TennisRacqu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

Commit message: Racquet attached

File: mmp_panda.urdf (robot description, URDF)
Before this commit: robot mmp_panda, 12 links, 10 joints
Links:
- link racquetlink: geometry visual mesh filename=../../../CS225a_TennisBot/Objects/Visual/TennisRacquet.obj
Joints:
- added joint joint8: type revolute, parent link7, child racquetlink, origin xyz=0.088 0 0 rpy=1.57079632679 0 0, axis 0 0 1, limit lower=-2.8973 upper=2.8973 effort=12 velocity=2.6100

Commit message: Changed racquet joint to fixed

File: mmp_panda.urdf (robot description, URDF)
Before this commit: robot mmp_panda, 12 links, 11 joints
Joints:
- joint joint8: type revolute -> fixed

Commit message: Added png images and made some adjustments to racquet and world urdf

File: mmp_panda.urdf (robot description, URDF)
Before this commit: robot mmp_panda, 12 links, 11 joints
Links:
- link link7: mass 3.0 -> 0.03268873

Commit message: Controller updates

File: mmp_panda.urdf (robot description, URDF)
Before this commit: robot mmp_panda, 12 links, 11 joints
Links:
- link racquetlink: geometry collision mesh filename=../../../CS225a_TennisBot/Objects/Visual/CollisionMeshRacqu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; visual mesh filename=../../../CS225a_TennisBot/Objects/Visual/TennisRacquet.obj

Commit message: Controller updates
Looking at converting world frame to robot frame, need to subtract world.urdf position

File: mmp_panda.urdf (robot description, URDF)
Before this commit: robot mmp_panda, 12 links, 11 joints
Links:
- link racquetlink: geometry collision mesh filename=../../../CS225a_TennisBot/Objects/Visual/TennisRacquet.obj; visual mesh filename=../../../CS225a_TennisBot/Objects/Visual/CollisionMeshRacqu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

Commit message: change mmp_panda velocity limit

File: mmp_panda.urdf (robot description, URDF)
Before this commit: robot mmp_panda, 12 links, 11 joints
Joints:
- joint base_prismatic_x: limit lower=-2.8973 upper=2.9873 effort=87 velocity=2.1750 -> effort=100 velocity=1000.0
- joint base_prismatic_y: limit lower=-2.8973 upper=2.9873 effort=87 velocity=2.1750 -> effort=100 velocity=1000.0

Commit message: in the middle of parameter tuning

File: mmp_panda.urdf (robot description, URDF)
Before this commit: robot mmp_panda, 12 links, 11 joints
Links:
- link racquetlink: geometry collision mesh filename=../../../CS225a_TennisBot/Objects/Visual/TennisRacquet.obj; visual mesh filename=../../../CS225a_TennisBot/Objects/Visual/TennisRacquet.obj

Commit message: Copy paste tennis launcher

File: mmp_panda.urdf (robot description, URDF)
Before this commit: robot mmp_panda, 12 links, 11 joints
Links:
- link racquetlink: geometry collision box size=0.25 1.5 0.0002; visual mesh filename=../../../CS225a_TennisBot/Objects/Visual/TennisRacquet.obj
Joints:
- joint joint8: origin xyz=0.088 0 0 rpy=1.57079632679 0 0 -> xyz=0.0 0 0 rpy=1.57079632679 0 0

Commit message: disabled interpolation, changed urdf

File: mmp_panda.urdf (robot description, URDF)
Before this commit: robot mmp_panda, 12 links, 11 joints
Joints:
- joint base_prismatic_x: limit effort=100 velocity=1000.0 -> effort=0 velocity=2.0
- joint base_prismatic_y: limit effort=100 velocity=1000.0 -> effort=0 velocity=2.0
- joint joint1: limit lower=-2.8973 upper=2.8973 effort=87 velocity=2.1750 -> lower=-2.8973 upper=2.8973 effort=100 velocity=100.0

Commit message: Test

File: mmp_panda.urdf (robot description, URDF)
Before this commit: robot mmp_panda, 12 links, 11 joints
Links:
- link racquetlink: geometry collision mesh filename=../../../CS225a_TennisBot/Objects/Visual/CollisionMeshRacqu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; visual mesh filename=../../../CS225a_TennisBot/Objects/Visual/CollisionMeshRacqu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

Commit message: small court final, working well

File: mmp_panda.urdf (robot description, URDF)
Before this commit: robot mmp_panda, 12 links, 11 joints
Links:
- link racquetlink: geometry collision box size=0.25 1.5 0.0002; visual mesh filename=../../../CS225a_TennisBot/Objects/Visual/TennisRacquet.obj
